Commit message: Fixed frame issues

File: ouster_backpack.urdf (robot description, URDF)
Before this commit: robot cartographer_backpack_3d, 3 links, 2 joints
Links:
- removed link os1_lidar
- added link os1; visual cylinder length=0.07 radius=0.05
Joints:
- joint os1_link_joint: child os1_lidar -> os1
